File: lux106_001/lux106_001.kicad_sch (KiCad schematic)
At the start: 14 parts

Commit message: update
Parts:
- removed R?: 100k, Resistor_THT:R_Axial_DIN0309_L9.0mm_D3.2mm_P2.54mm_Vertical, symbol pspice:R
- added BT1: Battery_Cell, TerminalBlock:TerminalBlock_Altech_AK300-2_P5.00mm, symbol Device:Battery_Cell
- added C1, C2, C3, C4: 22u, Capacitor_THT:CP_Radial_D5.0mm_P2.50mm, symbol Device:C_Polarized
- added R10, R2, R3, R5, R7, R8, R9: 100k, Resistor_THT:R_Axial_DIN0309_L9.0mm_D3.2mm_P2.54mm_Vertical, symbol pspice:R
- added R11, R12, R4, R6: R_Photo, Resistor_THT:R_Axial_DIN0204_L3.6mm_D1.6mm_P2.54mm_Vertical, symbol Device:R_Photo
- U2: renamed from U?; footprint (none) -> Package_DIP:DIP-14_W7.62mm_Socket
- U2: renamed from U?; footprint Package_DIP:DIP-8_W7.62mm_Socket -> Package_DIP:DIP-14_W7.62mm_Socket
- gave numbers to parts that had none: 1
Connections:
- net at R1.1: now also U2.5 (+)
- net at R1.2: now also U1.1, C1.1, R6.2
- net at U1.5: now also C2.1, R3.2, R4.2
- net at U1.6: now also R4.1
- net at U1.2: now also R6.1
- net at U2.10 (+): now also R9.1
- net at U2.8: now also R7.1
- net at U2.9 (-): now also R7.2
- net Earth: now reaches U2.11 (V-)
- net Earth: now also BT1.2 (-), C1.2, C2.2, C3.2, C4.2
- net VCC: now reaches U2.4 (V+)
- net VCC: now also BT1.1 (+)
- net at U1.8: now also R12.1
- net at U1.9: now also C4.1, R10.2, R12.2
- net at U2.12 (+): now also R10.1
- net at U2.13 (-): now also R8.2
- net at U2.14: now also R8.1
- net at U2.1: now also R2.1
- net at U2.2 (-): now also R2.2
- net at U2.3 (+): now also R3.1
- net at U2.6 (-): now also R5.2
- net at U2.7: now also R5.1
- net at U1.12: now also R11.1
- net at U1.13: now also C3.1, R11.2, R9.2
Other:
- moved on the sheet: R1, U1A, U1B, U1C, U1D, U1E, U1F, U1G, U2A, U2B, U2C, U2D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

Commit message: update
Parts:
- added D1: LED, LED_THT:LED_D5.0mm_Clear, symbol Device:LED
- added J1: Screw_Terminal_01x02, TerminalBlock:TerminalBlock_Altech_AK300-2_P5.00mm, symbol Connector:Screw_Terminal_01x02
- added R13: 1k, Resistor_THT:R_Axial_DIN0309_L9.0mm_D3.2mm_P2.54mm_Vertical, symbol Device:R
- U1: footprint DIP-14_W7.62mm_Socket -> Package_DIP:DIP-14_W7.62mm_Socket
- U1: footprint (none) -> Package_DIP:DIP-14_W7.62mm_Socket
Connections:
- net Earth: now also U1.7 (VSS), J1.1 (Pin_1), R13.1
- net VCC: now also U1.14 (VDD), D1.2 (A)
- net OUT: now reaches R2.1, U2.1
- net OUT: now also R5.1, R7.1, R8.1, U2.14, U2.7, U2.8, J1.2 (Pin_2)
- new net: D1.1 (K), R13.2

Commit message: update
Parts:
- added R14, R15, R16, R17: 1k, Resistor_THT:R_Axial_DIN0309_L9.0mm_D3.2mm_P2.54mm_Vertical, symbol pspice:R
Connections:
- net OUT: now also R14.1, R15.1, R16.1, R17.1; no longer R2.1, R5.1, R7.1, R8.1, U2.1, U2.14, U2.7, U2.8
- new net: R14.2, R2.1, U2.1
- new net: R16.2, R7.1, U2.8
- new net: R15.2, R5.1, U2.7
- new net: R17.2, R8.1, U2.14
Other:
- moved on the sheet: C3, C4, J1, R10, R11, R12, R7, R8, R9, U1D, U1F, U2C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
