File: lux106_002/lux106_002.kicad_pcb (KiCad board)
At the start: 2 copper layers, 48.3 x 68.6 mm, 29 parts, among them J1 Screw_Terminal_01x02, U1 40106, U2 LM324

Commit message: update
Parts:
- moved R10 1.66 mm to (111.8, 96.9)
Routing:
- net Net-(R10-Pad1): track 11.9 -> 13.8 mm
- net Net-(C4-Pad1): track 23.2 -> 21.5 mm
Changed lines of the file:
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@@
   )
   (footprint "Resistor_THT:R_Axial_DIN0309_L9.0mm_D3.2mm_P2.54mm_Vertical" (layer "F.Cu")
-    (at 110.85 98.22364 90)
+    (at 111.82138 96.878865 90)
     (descr "Resistor, Axial_DIN0309 series, Axial, Vertical, pin pitch=2.54mm, 0.5W = 1/2W, length*diameter=9*3.2mm^2, http://cdn-reichelt.de/documents/datenblatt/B400/1_4W%23YAG.pdf")
     (tags "Resistor Axial_DIN0309 series Axial Vertical pin pitch 2.54mm 0.5W = 1/2W length 9mm diameter 3.2mm")
@@
   (segment (start 105.08 76.19) (end 100.365 76.19) (width 0.25) (layer "F.Cu") (net 3))
   (segment (start 116.84 83.82) (end 116.84 99.06) (width 0.25) (layer "F.Cu") (net 3))
-  (segment (start 114.3 88.9) (end 114.3 92.23364) (width 0.25) (layer "F.Cu") (net 4))
-  (segment (start 111.76 86.36) (end 114.3 88.9) (width 0.25) (layer "F.Cu") (net 4))
   (segment (start 104.58 86.35) (end 111.76 86.35) (width 0.25) (layer "F.Cu") (net 4))
+  (segment (start 111.82138 94.338865) (end 114.3 91.860245) (width 0.25) (layer "F.Cu") (net 4))
   (segment (start 111.76 86.35) (end 111.76 86.36) (width 0.25) (layer "F.Cu") (net 4))
+  (segment (start 114.3 91.860245) (end 114.3 88.89) (width 0.25) (layer "F.Cu") (net 4))
   (segment (start 104.555 86.325) (end 104.58 86.35) (width 0.25) (layer "F.Cu") (net 4))
   (segment (start 100.34 86.325) (end 104.555 86.325) (width 0.25) (layer "F.Cu") (net 4))
-  (segment (start 114.3 92.23364) (end 110.85 95.68364) (width 0.25) (layer "F.Cu") (net 4))
+  (segment (start 114.3 88.89) (end 111.76 86.35) (width 0.25) (layer "F.Cu") (net 4))
   (segment (start 86.36 116.84) (end 86.36 113.36) (width 0.25) (layer "F.Cu") (net 5))
   (segment (start 92.695 111.76) (end 92.7 111.765) (width 0.25) (layer "F.Cu") (net 5))
@@
   (segment (start 111.755 106.685) (end 100.32 106.685) (width 0.25) (layer "F.Cu") (net 20))
   (segment (start 116.84 101.6) (end 111.755 106.685) (width 0.25) (layer "F.Cu") (net 20))
-  (segment (start 110.85 98.22364) (end 107.46864 101.605) (width 0.25) (layer "F.Cu") (net 21))
-  (segment (start 107.46864 101.605) (end 100.32 101.605) (width 0.25) (layer "F.Cu") (net 21))
+  (segment (start 111.82138 96.878865) (end 107.095245 101.605) (width 0.25) (layer "F.Cu") (net 21))
+  (segment (start 111.82138 96.58138) (end 111.76 96.52) (width 0.25) (layer "F.Cu") (net 21))
+  (segment (start 111.82138 96.878865) (end 111.82138 96.58138) (width 0.25) (layer "F.Cu") (net 21))
+  (segment (start 107.095245 101.605) (end 100.32 101.605) (width 0.25) (layer "F.Cu") (net 21))
   (segment (start 105.055 78.705) (end 105.08 78.73) (width 0.25) (layer "F.Cu") (net 22))
   (segment (start 100.34 78.705) (end 105.055 78.705) (width 0.25) (layer "F.Cu") (net 22))

Commit message: fix version 1.0
Parts:
- moved BT1 2.55 mm to (114.3, 63.6)
- moved ? 1.88 mm to (116.8, 124.5)
- moved R6 1.60 mm to (88.9, 76.2)
- moved C1 1.04 mm to (82.3, 73.7)
Routing:
- net Earth: track 130.6 -> 127.0 mm
- net VCC: track 67.1 -> 64.6 mm
- net Net-(R6-Pad1): track 5.44 -> 3.84 mm
- net Net-(C1-Pad1): track 31.0 -> 30.3 mm
Other:
- board size 48.3 x 68.6 mm -> 48.3 x 71.1 mm
- board text added: "LUXCHORD 1.0 franeum 2023.11"
