File: lux106_1_1/lux106_1_1.kicad_pcb (KiCad board)
At the start: 2 copper layers, 68.6 x 88.9 mm, 35 parts, among them J1 Screw_Terminal_01x02, SW1 SW_DPST_x2, U1 40106, U2 LM324

Commit message: update v1.1
Parts:
- removed SW1: SW_DPST_x2, Button_Switch_THT:SW_DIP_SPSTx01_Slide_6.7x4.1mm_W7.62mm_P2.54mm_LowProfile
- added RV5: R_Potentiometer, Potentiometer_THT:Potentiometer_Alps_RK097_Single_Horizontal, F.Cu at (81.3, 127.0)
- added SW2: SW_SPDT, Daisy_Electrosmith:mini_SPDT_switch, F.Cu at (138.4, 72.4)
- R1, R2, R3, R4: value 1K -> 100
- moved R10 14.7 mm to (87.6, 78.1)
- moved R5 10.5 mm to (121.9, 68.6), turned to 0 degrees
- moved SCRW 1 9.25 mm to (90.2, 132.1)
- moved R2 8.14 mm to (87.6, 73.7), turned to 0 degrees
- moved RV3 7.66 mm to (81.3, 109.2)
- moved R15 7.39 mm to (106.7, 119.4)
- moved R6 7.33 mm to (88.9, 97.2)
- moved R14 6.76 mm to (106.7, 89.5)
- moved R16 6.76 mm to (106.7, 108.6)
- moved U2 6.13 mm to (101.6, 105.4)
- moved J1 5.68 mm to (104.1, 132.1)
- moved C6 5.39 mm to (96.5, 124.5), turned to 180 degrees
- moved RV4 5.08 mm to (81.3, 91.5)
- moved R7 4.63 mm to (92.1, 85.7)
- moved R8 4.22 mm to (100.3, 85.7)
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Connections:
- C6 pad 2: OUT -> Net-(C6-Pad2)
Routing:
- net Net-(R10-Pad1): track 26.6 -> 44.7 mm
- net Net-(C6-Pad2): track 0.00 -> 14.8 mm
- net OUT: track 22.2 -> 33.6 mm
- net Net-(C1-Pad1): track 40.7 -> 52.1 mm
- net Net-(R3-Pad1): track 58.4 -> 48.5 mm
- net Net-(U2C-+): track 14.4 -> 5.87 mm
- net Net-(C2-Pad1): track 37.9 -> 32.3 mm
- net Net-(R2-Pad1): track 12.7 -> 7.40 mm
- net Net-(R4-Pad1): track 65.1 -> 59.9 mm
- net Net-(U2C--): track 5.70 -> 10.5 mm
- net Net-(C4-Pad1): track 73.6 -> 69.0 mm
- net Net-(C3-Pad1): track 71.7 -> 67.0 mm
- net Net-(U2D--): track 9.00 -> 5.87 mm
- net Net-(R16-Pad1): track 8.89 -> 11.9 mm
- net GND: track 143.5 -> 140.8 mm
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- added copper zone on B.Cu, net (none)
- added copper zone on F.Cu, net (none)
Other:
- board size 68.6 x 88.9 mm -> 68.6 x 85.1 mm
- board text added: "+"
- board text added: "-"
