File: lux106_1_1/lux106_1_1.kicad_sch (KiCad schematic)
At the start: 33 parts, among them J1 Screw_Terminal_01x02, SW1 SW_DPST_x2, U1 40106, U2 LM324

Commit message: update v1.1
Parts:
- removed SW1: SW_DPST_x2, Button_Switch_THT:SW_DIP_SPSTx01_Slide_6.7x4.1mm_W7.62mm_P2.54mm_LowProfile, symbol Switch:SW_DPST_x2
- added RV5: R_Potentiometer, Potentiometer_THT:Potentiometer_Alps_RK097_Single_Horizontal, symbol Device:R_Potentiometer
- added SW2: SW_SPDT, Daisy_Electrosmith:mini_SPDT_switch, symbol Switch:SW_SPDT
- R1, R2, R3, R4: value 1K -> 100
Connections:
- net GND: now also SW2.1 (A)
- net OUT: now also RV5.3; no longer C6.2
- net at BT1.2 (-), C5.2: now also SW2.2 (B)
- new net: C6.2, RV5.2
- no-connect marks 8 -> 10
Other:
- moved on the sheet: C6, D1, J1, R5, U1G
